File: attiny1614.sch (KiCad schematic (older format))
At the start: 12 parts, among them J1 Conn_01x07, J2 Conn_01x07, J3 Power, J4 UPDI, U1 AP7381-50SA, U2 ATtiny1614-SS

Commit message: gerbers and layout
Parts:
- removed J3: Power, Connector_PinHeader_1.27mm:PinHeader_1x02_P1.27mm_Vertical, symbol Connector_Generic:Conn_01x02
- removed U1: AP7381-50SA, Package_TO_SOT_SMD:SOT-23, symbol attiny1614-rescue:AP7381-50SA-Regulator_Linear
- added D2: BAT54CW, Package_TO_SOT_SMD:SOT-323_SC-70, symbol Diode:BAT54CW
- added JP1: VCC Select, Connector_PinHeader_1.27mm:PinHeader_1x03_P1.27mm_Vertical, symbol Jumper:Jumper_3_Bridged12
- added R1: 100R, Resistor_SMD:R_0603_1608Metric_Pad1.05x0.95mm_HandSolder, symbol Device:R_Small
- added R2, R3: 10K, Resistor_SMD:R_0603_1608Metric_Pad1.05x0.95mm_HandSolder, symbol Device:R_Small
- added SW1: Reset, Button_Switch_SMD:SW_Push_SPST_NO_Alps_SKRK, symbol Switch:SW_Push
- added U2: AP7381-33SA, Package_TO_SOT_SMD:SOT-23, symbol Regulator_Linear:AP7381-33SA
- J1: renamed from J4; footprint Connector_PinHeader_1.27mm:PinHeader_2x03_P1.27mm_Vertical -> Connector_PinHeader_1.27mm:PinHeader_1x03_P1.27mm_Vertical; symbol Connector_Generic:Conn_02x03_Odd_Even -> Connector_Generic:Conn_01x03
- renumbered J1 to J2, J2 to J3, R1 to R4, R2 to R5, U2 to U1
Connections:
- net labels added: MISO, MOSI, RXD, SCA, SCK, SCL, TXD
- net labels removed: 5V, PA1, PA2, PA3, PB0, PB1, PB2, PB3
- wire segments 54 -> 71
- no-connect marks 3 -> 0
Other:
- moved on the sheet: C1, C2, C3, D1, J2, J3, R4, R5, U1
